Commit message: modified:   hb_task1b_ws/README.md 	modified:   hb_task1b_ws/src/hb_task_1b/urdf/hb_bot.urdf.xacro

File: hb_task1b_ws/src/hb_task_1b/urdf/hb_bot.urdf.xacro (robot description, xacro)
@@ -91,5 +91,71 @@
         </visual>
     </link>
-    <!-- Joint -->
+    <!-- front_wheel -->
+    <link name ="front_wheel">
+        <inertial>
+            <origin
+                xyz="0.0 -0.05 0.0"
+                rpy="1.57 0 0" />
+            <mass
+                value="0.060" />
+            <inertia
+                ixx="1.825e-4"
+                ixy="0"
+                ixz="0.00000000"
+                iyy="1.825e-4"
+                iyz="0"
+                izz="1.825e-4" />
+        </inertial>
+         <collision name="F_collision">
+         <origin
+                xyz="0 -0.05 0.0"
+                rpy="1.57 0 0" />
+          <geometry>
+            <cylinder length="0.13" radius="0.14"/>
+          </geometry>
+        </collision>
+        <visual>
+            <origin
+            xyz="0.0 0.0 0.0"
+            rpy="0.0 0.0 0.0" />
+            <geometry>
+                <mesh filename ="file://$(find hb_task_1b)/meshes/wheel.stl" scale="5 5 5"/>
+            </geometry>
+        </visual>
+    </link>
+    <!-- left_wheel -->
+    <link name ="left_wheel">
+        <inertial>
+            <origin
+                xyz="0 -0.05 0.0"
+                rpy="1.57 0 0" />
+            <mass
+                value="0.060" />
+            <inertia
+                ixx="1.825e-4"
+                ixy="0"
+                ixz="0.00000000"
+                iyy="1.825e-4"
+                iyz="0"
+                izz="1.825e-4" />
+        </inertial>
+         <collision name="L_collision">
+         <origin
+                xyz="0 -0.05 0.0"
+                rpy="1.57 0 0" />
+          <geometry>
+            <cylinder length="0.13" radius="0.14"/>
+          </geometry>
+        </collision>
+        <visual>
+            <origin
+            xyz="0.0 0.0 0.0"
+            rpy="0.0 0.0 0.0" />
+            <geometry>
+                <mesh filename ="file://$(find hb_task_1b)/meshes/wheel.stl" scale="5 5 5"/>
+            </geometry>
+        </visual>
+    </link>
+    <!-- right_joint -->
     <joint name ="right_wheel_joint" type="continuous" >
         <origin
@@ -103,7 +169,47 @@
             velocity="5" />
     </joint>
+    <!-- front_joint -->
+    <joint name ="front_wheel_joint" type="continuous" >
+        <origin
+                xyz="-0.57 -0.34 0.18"
+                rpy="0 0 2.1" />
+        <parent link="base_link"/>
+        <child link="front_wheel"/>
+        <axis xyz="0.0 1.0 0.0"/>
+         <limit
+            effort="5"
+            velocity="5" />
+    </joint>
+    <!-- left_joint -->
+    <joint name ="left_wheel_joint" type="continuous" >
+        <origin
+                xyz="0.50 -0.31 0.16"
+                rpy="0 0 1.05" />
+        <parent link="base_link"/>
+        <child link="left_wheel"/>
+        <axis xyz="0.0 1.0 0.0"/>
+         <limit
+            effort="5"
+            velocity="5" />
+    </joint>
     <!-- material properties -->
     <gazebo reference="right_wheel">
         <material>Gazebo/Black</material>
     </gazebo>
+    <gazebo reference="front_wheel">
+        <material>Gazebo/Black</material>
+    </gazebo>
+    <gazebo reference="left_wheel">
+        <material>Gazebo/Black</material>
+    </gazebo>
+    <!-- ros_control plugin -->
+  <gazebo>
+    <plugin name="object_controller" filename="libgazebo_ros_planar_move.so">
+      <commandTopic>cmd_vel</commandTopic>
+      <odometryTopic>odom</odometryTopic>
+      <odometryFrame>odom</odometryFrame>
+      <odometryRate>20.0</odometryRate>
+      <robotBaseFrame>chasis</robotBaseFrame>
+    </plugin>
+  </gazebo>
 </robot>
